Commit message: Modified m2wr_descrition to one-kinect-robot

File: files/catkin_ws/src/one-kinect-robot/urdf/kinect-robot.xacro (robot description, xacro)
@@ -1,7 +1,7 @@
 <?xml version="1.0" ?>
-<robot name="m2wr" xmlns:xacro="http://www.ros.org/wiki/xacro">
-  <xacro:include filename="$(find m2wr_description)/urdf/materials.xacro" />
-  <xacro:include filename="$(find m2wr_description)/urdf/m2wr.gazebo" />
-  <xacro:include filename="$(find m2wr_description)/urdf/macros.xacro" />
+<robot name="kinect-robot" xmlns:xacro="http://www.ros.org/wiki/xacro">
+  <xacro:include filename="$(find one-kinect-robot)/urdf/materials.xacro" />
+  <xacro:include filename="$(find one-kinect-robot)/urdf/kinect-robot.gazebo" />
+  <xacro:include filename="$(find one-kinect-robot)/urdf/macros.xacro" />
   <link name="link_chassis">
     <!-- pose and inertial -->
@@ -49,14 +49,14 @@
     </visual>
   </link>
-  <link name="sensor_laser">
+  <link name="kinect_sensor">
     <inertial>
         <origin xyz="0 0 0" rpy="0 0 0" />
         <mass value="1" />
-        <xacro:cylinder_inertia mass="1" r="0.05" l="0.1" />
+        <xacro:cube_inertia mass="1" w="0.05" h="0.05" d="0.05" />
     </inertial>
     <visual>
         <origin xyz="0 0 0" rpy="0 0 0" />
         <geometry>
-        <cylinder radius="0.05" length="0.1"/>
+          <box size="0.05 0.05 0.05"/>
         </geometry>
         <material name="white" />
@@ -65,12 +65,12 @@
         <origin xyz="0 0 0" rpy="0 0 0"/>
         <geometry>
-        <cylinder radius="0.05" length="0.1"/>
+          <box size="0.05 0.05 0.05"/>
         </geometry>
     </collision>
   </link>
-  <joint name="joint_sensor_laser" type="fixed">
+  <joint name="joint_kinect_sensor" type="fixed">
     <origin xyz="0.15 0 0.05" rpy="0 0 0"/>
     <parent link="link_chassis"/>
-    <child link="sensor_laser"/>
+    <child link="kinect_sensor"/>
   </joint>
   <xacro:link_wheel name="link_right_wheel" />

File: files/catkin_ws/src/one-kinect-robot/urdf/macros.xacro (robot description, xacro)
@@ -32,4 +32,9 @@
       </joint>
     </macro>
+    <macro name="cube_inertia" params="mass w h d">
+      <inertia  ixx="${mass*(h*h+d*d)/12}" ixy = "0" ixz = "0"
+            iyy="${mass*(w*w+d*d)/12}" iyz = "0"
+            izz="${mass*(w*w+h*h)/12}" />
+    </macro>
     <macro name="cylinder_inertia" params="mass r l">
       <inertia  ixx="${mass*(3*r*r+l*l)/12}" ixy = "0" ixz = "0"
