Commit message: Updating files - Docker now includes URG-NODE

File: files/catkin_ws/src/m2wr_description/urdf/m2wr.xacro (robot description, xacro)
@@ -49,28 +49,8 @@
     </visual>
   </link>
-  <link name="sensor_laser">
-    <inertial>
-        <origin xyz="0 0 0" rpy="0 0 0" />
-        <mass value="1" />
-        <xacro:cylinder_inertia mass="1" r="0.05" l="0.1" />
-    </inertial>
-    <visual>
-        <origin xyz="0 0 0" rpy="0 0 0" />
-        <geometry>
-        <cylinder radius="0.05" length="0.1"/>
-        </geometry>
-        <material name="white" />
-    </visual>
-    <collision>
-        <origin xyz="0 0 0" rpy="0 0 0"/>
-        <geometry>
-        <cylinder radius="0.05" length="0.1"/>
-        </geometry>
-    </collision>
-  </link>
-  <joint name="joint_sensor_laser" type="fixed">
-    <origin xyz="0.15 0 0.05" rpy="0 0 0"/>
-    <parent link="link_chassis"/>
-    <child link="sensor_laser"/>
+  <joint name="laser_joint" type="fixed">
+    <origin xyz="0.15 0 0.05" rpy="0 0 0" />
+    <parent link="link_chassis" />
+    <child link="laser" />
   </joint>
   <xacro:link_wheel name="link_right_wheel" />

Commit message: LIDAR and mapping fully operational.

File: files/catkin_ws/src/m2wr_description/urdf/m2wr.xacro (robot description, xacro)
@@ -4,4 +4,5 @@
   <xacro:include filename="$(find m2wr_description)/urdf/m2wr.gazebo" />
   <xacro:include filename="$(find m2wr_description)/urdf/macros.xacro" />
+  <!-- <xacro:include filename="$(find m2wr_description)/urdf/lidar.xacro"/> -->
   <link name="link_chassis">
     <!-- pose and inertial -->
@@ -49,9 +50,34 @@
     </visual>
   </link>
-  <joint name="laser_joint" type="fixed">
-    <origin xyz="0.15 0 0.05" rpy="0 0 0" />
-    <parent link="link_chassis" />
-    <child link="laser" />
+  <link name="sensor_laser">
+    <inertial>
+        <origin xyz="0 0 0" rpy="0 0 0" />
+        <mass value="1" />
+        <xacro:cylinder_inertia mass="1" r="0.05" l="0.1" />
+    </inertial>
+    <visual>
+        <origin xyz="0 0 0" rpy="0 0 0" />
+        <geometry>
+        <cylinder radius="0.05" length="0.1"/>
+        </geometry>
+        <material name="white" />
+    </visual>
+    <collision>
+        <origin xyz="0 0 0" rpy="0 0 0"/>
+        <geometry>
+        <cylinder radius="0.05" length="0.1"/>
+        </geometry>
+    </collision>
+    </link>
+  <joint name="joint_sensor_laser" type="fixed">
+    <origin xyz="0.15 0 0.05" rpy="0 0 0"/>
+    <parent link="link_chassis"/>
+    <child link="sensor_laser"/>
   </joint>
+  <!--<joint name="joint_sensor_kinect" type="fixed">
+    <origin xyz="0.15 0 0.3" rpy="0 0 0"/>
+    <parent link="link_chassis"/>
+    <child link="sensor_kinect"/>
+  </joint>-->
   <xacro:link_wheel name="link_right_wheel" />
   <xacro:joint_wheel name="joint_right_wheel" child="link_right_wheel" origin_xyz="-0.05 0.15 0" />
